Commit message: feat: 增加雷达与深度相机仿真及感知测试方案

File: src/ackermann_line_following_description/urdf/ackermann_car.urdf.xacro (robot description, xacro)
@@ -213,4 +213,45 @@
     </sensor>
   </gazebo>
+  <!-- 感知相机水平朝前；光学坐标为右、下、前。 -->
+  <link name="rgbd_link"/>
+  <joint name="rgbd_joint" type="fixed">
+    <parent link="base_link"/><child link="rgbd_link"/>
+    <origin xyz="0.36 0 0.25"/>
+  </joint>
+  <link name="rgbd_optical_frame"/>
+  <joint name="rgbd_optical_joint" type="fixed">
+    <parent link="rgbd_link"/><child link="rgbd_optical_frame"/>
+    <origin rpy="${-pi_value/2} 0 ${-pi_value/2}"/>
+  </joint>
+  <link name="lidar_link"/>
+  <joint name="lidar_joint" type="fixed">
+    <parent link="base_link"/><child link="lidar_link"/>
+    <origin xyz="0 0 0.36"/>
+  </joint>
+  <gazebo reference="lidar_link">
+    <sensor name="lidar" type="gpu_lidar">
+      <gz_frame_id>lidar_link</gz_frame_id>
+      <topic>/scan</topic><always_on>true</always_on><update_rate>10</update_rate>
+      <lidar>
+        <scan><horizontal><samples>720</samples><resolution>1</resolution>
+          <min_angle>${-pi_value}</min_angle><max_angle>${pi_value}</max_angle>
+        </horizontal></scan>
+        <range><min>0.12</min><max>12</max><resolution>0.01</resolution></range>
+        <noise><type>gaussian</type><mean>0</mean><stddev>0.01</stddev></noise>
+      </lidar>
+    </sensor>
+  </gazebo>
+  <gazebo reference="rgbd_link">
+    <sensor name="rgbd" type="rgbd_camera">
+      <gz_frame_id>rgbd_optical_frame</gz_frame_id>
+      <topic>/rgbd</topic><always_on>true</always_on><update_rate>15</update_rate>
+      <camera>
+        <horizontal_fov>1.211</horizontal_fov>
+        <image><width>640</width><height>480</height><format>R8G8B8</format></image>
+        <clip><near>0.2</near><far>8</far></clip>
+        <depth_camera><clip><near>0.2</near><far>8</far></clip></depth_camera>
+      </camera>
+    </sensor>
+  </gazebo>
   <!-- Gazebo Sim's native Ackermann system is model-name agnostic at runtime. -->
   <gazebo>

Commit message: feat: add sim-to-real control and EKF path

File: src/ackermann_line_following_description/urdf/ackermann_car.urdf.xacro (robot description, xacro)
@@ -230,4 +230,29 @@
     <origin xyz="0 0 0.36"/>
   </joint>
+  <link name="imu_link"/>
+  <joint name="imu_joint" type="fixed">
+    <parent link="base_link"/><child link="imu_link"/>
+    <origin xyz="0 0 0.08"/>
+  </joint>
+  <gazebo reference="imu_link">
+    <sensor name="imu" type="imu">
+      <gz_frame_id>imu_link</gz_frame_id>
+      <topic>/imu/data_raw</topic>
+      <always_on>true</always_on>
+      <update_rate>100</update_rate>
+      <imu>
+        <angular_velocity>
+          <x><noise type="gaussian"><mean>0</mean><stddev>0.002</stddev></noise></x>
+          <y><noise type="gaussian"><mean>0</mean><stddev>0.002</stddev></noise></y>
+          <z><noise type="gaussian"><mean>0</mean><stddev>0.002</stddev></noise></z>
+        </angular_velocity>
+        <linear_acceleration>
+          <x><noise type="gaussian"><mean>0</mean><stddev>0.03</stddev></noise></x>
+          <y><noise type="gaussian"><mean>0</mean><stddev>0.03</stddev></noise></y>
+          <z><noise type="gaussian"><mean>0</mean><stddev>0.03</stddev></noise></z>
+        </linear_acceleration>
+      </imu>
+    </sensor>
+  </gazebo>
   <gazebo reference="lidar_link">
     <!--
